File: multicomp/NASCOM4/kicad/nascom_ng/nascom_ng_fdc.sch (KiCad schematic (older format))
At the start: 24 parts, among them J11 Conn_02x02_Odd_Even, J13 Conn_02x02_Odd_Even, J7 Conn_02x17_Odd_Even, U14 74LS38, U15 74LS174, U2 WD2797, U3 74LS06, U8 74LS367, U9 74HCT123

Commit message: All nets routed, ref designators resequenced, nearly finished!
Parts:
- renumbered C4 to C10, C3 to C14, C1 to C21, C2 to C22, D4 to D7, J11 to J10, J13 to J4, J7 to J8, R17 to R11, R13 to R12, R15 to R13, R12 to R14, R14 to R15, R18 to R16, R16 to R20, RV2 to RV1, RV1 to RV2, U9 to U10, U8 to U11, U2 to U13, U15 to U14, U3 to U15, U14 to U17
Connections:
- net GND: no longer J4.4 (Pin_4)
- no-connect marks 6 -> 7
Other:
- note added: "DRIVE PIN 6 PIN 34\nTeac FD-55 Drive select 3 READY\nPertec FD250 Drive select 3 unused\nMicropolis 1015 READY Drive select 3\n\nUse "L5 (DISK READY)" to route READY or to select internal\nREADY generation"
- note added: "Write precompensation\nNo link: always\n1-2: never\n1-3: for track>43"
- note removed: ""L9 (WRPRECOMP)""
- note removed: "DRIVE PIN 6 PIN 34\nTeac FD-55 Drive select 3 READY\nPertec FD250 Drive select 3 unused\nMicropolis 1015 READY Drive select 3\n\nUse jumpers to route READY or to select internal\nREADY generation"

Commit message: Files for REV A release to PCB manufacture
Parts:
- renumbered C10 to C12, C14 to C15, C22 to C24, C21 to C25, J8 to J20, J4 to J5
Other:
- note removed: "TODO can I push all of this back into the FPGA"
Changed lines of the file:
@@
 	1250 1750 1050 1750
 $Comp
-L Device:CTRIM C21
+L Device:CTRIM C25
 U 1 1 5FDBD149
 P 1500 2850
-F 0 "C21" H 1616 2896 50  0000 L CNN
+F 0 "C25" H 1616 2896 50  0000 L CNN
 F 1 "5-65p" H 1616 2805 50  0000 L CNN
 F 2 "mylib:Trimmer_Vishay_BFC2808_Fig2" H 1500 2850 50  0001 C CNN
@@
 Out to FDD
 $Comp
-L Device:C C22
+L Device:C C24
 U 1 1 604E3959
 P 3750 2500
-F 0 "C22" V 3498 2500 50  0000 C CNN
+F 0 "C24" V 3498 2500 50  0000 C CNN
 F 1 "0.22u" V 3589 2500 50  0000 C CNN
 F 2 "Capacitor_THT:C_Disc_D7.5mm_W2.5mm_P5.00mm" H 3788 2350 50  0001 C CNN
@@
 $EndComp
 $Comp
-L Device:C C14
+L Device:C C15
 U 1 1 605EA818
 P 5650 3650
-F 0 "C14" H 5535 3604 50  0000 R CNN
+F 0 "C15" H 5535 3604 50  0000 R CNN
 F 1 "33p" H 5535 3695 50  0000 R CNN
 F 2 "Capacitor_THT:C_Disc_D3.0mm_W2.0mm_P2.50mm" H 5688 3500 50  0001 C CNN
@@
 	5650 4900 6150 4900
 $Comp
-L Device:CP_Small C10
+L Device:CP_Small C12
 U 1 1 6064BFF0
 P 5650 5100
-F 0 "C10" H 5738 5146 50  0000 L CNN
+F 0 "C12" H 5738 5146 50  0000 L CNN
 F 1 "1u" H 5738 5055 50  0000 L CNN
 F 2 "Capacitor_THT:CP_Radial_Tantal_D4.5mm_P5.00mm" H 5650 5100 50  0001 C CNN
@@
 Text GLabel 1100 6350 0    50   Input ~ 0
 D5_5V
-Text Notes 8950 6400 0    50   ~ 0
-TODO can I push all of this back into the FPGA
 Text GLabel 1100 6550 0    50   Input ~ 0
 PORTE4_WR_5V
@@
 DRQ_5V
 $Comp
-L Connector_Generic:Conn_02x02_Odd_Even J4
+L Connector_Generic:Conn_02x02_Odd_Even J5
 U 1 1 6176BCD8
 P 3300 4400
-F 0 "J4" H 3350 4617 50  0000 C CNN
+F 0 "J5" H 3350 4617 50  0000 C CNN
 F 1 "Conn_02x02_Odd_Even" H 3350 4526 50  0000 C CNN
 F 2 "Connector_PinHeader_2.54mm:PinHeader_2x02_P2.54mm_Vertical" H 3300 4400 50  0001 C CNN
@@
 	9150 2800 8950 2800
 $Comp
-L Connector_Generic:Conn_02x17_Odd_Even J8
+L Connector_Generic:Conn_02x17_Odd_Even J20
 U 1 1 5FDA5F50
 P 9350 3600
-F 0 "J8" H 9400 4617 50  0000 C CNN
+F 0 "J20" H 9400 4617 50  0000 C CNN
 F 1 "Conn_02x17_Odd_Even" H 9400 4526 50  0000 C CNN
 F 2 "Connector_IDC:IDC-Header_2x17_P2.54mm_Vertical" H 9350 3600 50  0001 C CNN
